Commit message: Arucos funcionales en simulacion

File: src/description/urdf/lifter.urdf.xacro (robot description, xacro)
@@ -146,5 +146,5 @@
     <parent link="mast_inner_link"/>
     <child  link="cam_holder_link"/>
-    <origin xyz="0 0 0.105" rpy="0.7854 0 0"/>
+    <origin xyz="0 0 0.105" rpy="0.3491 0 0"/>  <!-- tilt camara 20deg hacia abajo (antes 45deg=0.7854) -->
   </joint>
   <!-- Camera: fixed to pan holder, sits on top of bracket

File: src/description/urdf/puzzlebot_gazebo.xacro (robot description, xacro)
@@ -65,5 +65,5 @@
         <image>
           <width>640</width>
-          <height>480</height>
+          <height>360</height>
           <format>R8G8B8</format>
         </image>

File: src/description/urdf/puzzlebot_with_lifter.urdf.xacro (robot description, xacro)
@@ -362,5 +362,5 @@
     <parent link="mast_inner_link"/>
     <child  link="cam_holder_link"/>
-    <origin xyz="0 0 0.105" rpy="0.7854 0 0"/>
+    <origin xyz="0 0 0.105" rpy="0.3491 0 0"/>  <!-- tilt camara 20deg hacia abajo (antes 45deg=0.7854) -->
   </joint>
   <!-- Camera: fixed to the pan holder, sits on top of bracket
